File: CellarRemote/CellarRemote.brd (EAGLE design)
At the start: 30.5 x 38.1 mm, 19 parts, among them M1 BSS84

Commit message: Minor updates to CellarRemote
Routing:
- net VCC: track 80.6 -> 95.4 mm
Other:
- board text added: "v1.1"
- board text removed: "v1.0"
Changed lines of the file:
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@@
 <text x="16.51" y="31.75" size="1.016" layer="22" ratio="15" rot="MR0">1WR</text>
 <text x="17.78" y="6.35" size="1.016" layer="22" ratio="15" rot="MR0">1WR</text>
-<text x="4.445" y="13.97" size="1.016" layer="22" ratio="15" rot="MR0">v1.0</text>
-<text x="1.27" y="15.24" size="1.016" layer="21" ratio="15">v1.0</text>
+<text x="4.445" y="13.97" size="1.016" layer="22" ratio="15" rot="MR0">v1.1</text>
+<text x="1.27" y="15.24" size="1.016" layer="21" ratio="15">v1.1</text>
 </plain>
 <attributes>
@@
 <wire x1="13.716" y1="27.94" x2="12.192" y2="26.416" width="0.4064" layer="1"/>
 <wire x1="12.192" y1="26.416" x2="5.08" y2="26.416" width="0.4064" layer="1"/>
-<wire x1="13.716" y1="27.94" x2="21.59" y2="27.94" width="0" layer="19" extent="1-1"/>
+<wire x1="21.59" y1="27.94" x2="21.59" y2="29.21" width="0.4064" layer="1"/>
+<wire x1="21.59" y1="29.21" x2="20.32" y2="30.48" width="0.4064" layer="1"/>
+<wire x1="20.32" y1="30.48" x2="13.97" y2="30.48" width="0.4064" layer="1"/>
+<wire x1="13.97" y1="30.48" x2="10.16" y2="34.29" width="0.4064" layer="1"/>
 </signal>
 <signal name="GND">
