File: modules/ext_i2c.brd (EAGLE design)
At the start: 25.4 x 17.7 mm, 11 parts, among them J1 MOLEX_MINILITE_TRAP_2, J2 MOLEX_MINILITE_TRAP_2, J3 MOLEX_MINILITE_TRAP_2, J4 1X06_HEADER_L1X06_EDGE_L, J5 1X06_HEADER_R1X06_EDGE_R, U1 P82B715D

Commit message: Minor changes to cellar controller. Rework of ext_i2c board
Parts:
- moved J4 1.27 mm to (1.27, 2.54)
- moved J5 1.27 mm to (24.1, 2.54)
- moved J1 0.25 mm to (6.60, 3.30)
- moved C1 0.25 mm to (12.4, 4.83)
Routing:
- net N$3: track 37.1 -> 33.3 mm
- net N$2: track 37.3 -> 33.5 mm
- net GND: track 2.54 -> 6.08 mm
- net 12V: track 26.0 -> 23.3 mm
- net N$1: track 25.4 -> 22.9 mm
- net 3.3V: track 45.2 -> 42.9 mm
Changed lines of the file:
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@@
 <layer number="230" name="230bmp" color="7" fill="1" visible="yes" active="yes"/>
 <layer number="231" name="231bmp" color="7" fill="1" visible="yes" active="yes"/>
+<layer number="232" name="Eagle3D_PG2" color="7" fill="1" visible="no" active="no"/>
+<layer number="233" name="Eagle3D_PG3" color="7" fill="1" visible="no" active="no"/>
 <layer number="248" name="Housing" color="7" fill="1" visible="yes" active="yes"/>
 <layer number="249" name="Edge" color="7" fill="1" visible="yes" active="yes"/>
@@
 </autorouter>
 <elements>
-<element name="J1" library="Puffin" package="MOLEX_MINILITE_TRAP_2" value="MOLEX_MINILITE_TRAP_2" x="6.35" y="3.302" smashed="yes" rot="R180">
-<attribute name="NAME" x="11.676" y="1.218" size="1.016" layer="21" font="vector" ratio="15" rot="R180"/>
+<element name="J1" library="Puffin" package="MOLEX_MINILITE_TRAP_2" value="MOLEX_MINILITE_TRAP_2" x="6.604" y="3.302" smashed="yes" rot="R180">
+<attribute name="NAME" x="11.93" y="1.218" size="1.016" layer="21" font="vector" ratio="15" rot="R180"/>
 </element>
 <element name="J2" library="Puffin" package="MOLEX_MINILITE_TRAP_2" value="MOLEX_MINILITE_TRAP_2" x="18.542" y="3.302" smashed="yes">
@@
 <attribute name="NAME" x="14.978" y="17.22" size="1.016" layer="21" font="vector" ratio="15" rot="R180"/>
 </element>
-<element name="J4" library="Puffin" package="1X06_EDGE_L" value="1X06_HEADER_L1X06_EDGE_L" x="0" y="2.54" smashed="yes">
-<attribute name="NAME" x="0.9398" y="16.3068" size="1.016" layer="25" font="vector" ratio="15"/>
-</element>
-<element name="J5" library="Puffin" package="1X06_EDGE_R" value="1X06_HEADER_R1X06_EDGE_R" x="25.4" y="2.54" smashed="yes">
-<attribute name="NAME" x="23.0378" y="16.3068" size="1.016" layer="25" font="vector" ratio="15"/>
+<element name="J4" library="Puffin" package="1X06_EDGE_L" value="1X06_HEADER_L1X06_EDGE_L" x="1.27" y="2.54" smashed="yes">
+<attribute name="NAME" x="2.2098" y="16.3068" size="1.016" layer="25" font="vector" ratio="15"/>
+</element>
+<element name="J5" library="Puffin" package="1X06_EDGE_R" value="1X06_HEADER_R1X06_EDGE_R" x="24.13" y="2.54" smashed="yes">
+<attribute name="NAME" x="21.7678" y="16.3068" size="1.016" layer="25" font="vector" ratio="15"/>
 </element>
 <element name="R1" library="resistor" package="R0805" value="2.2k" x="4.064" y="9.398" smashed="yes" rot="R90">
@@
 <attribute name="NAME" x="11.7602" y="12.5476" size="1.016" layer="25" font="vector" ratio="15" rot="SR270"/>
 </element>
-<element name="C1" library="SparkFun-Capacitors" package="0603-CAP" value="1.0uF" x="12.192" y="4.826" smashed="yes" rot="R270">
-<attribute name="PROD_ID" value="CAP-00868" x="12.192" y="4.826" size="1.778" layer="27" rot="R270" display="off"/>
-<attribute name="NAME" x="12.954" y="6.223" size="1.016" layer="25" font="vector" ratio="15" rot="R270"/>
+<element name="C1" library="SparkFun-Capacitors" package="0603-CAP" value="1.0uF" x="12.446" y="4.826" smashed="yes" rot="R270">
+<attribute name="PROD_ID" value="CAP-00868" x="12.446" y="4.826" size="1.778" layer="27" rot="R270" display="off"/>
+<attribute name="NAME" x="13.208" y="6.223" size="1.016" layer="25" font="vector" ratio="15" rot="R270"/>
 </element>
 </elements>
@@
 <contactref element="J4" pad="6"/>
 <contactref element="J5" pad="6"/>
-<wire x1="25.4" y1="15.24" x2="0" y2="15.24" width="0.8128" layer="16"/>
+<wire x1="24.13" y1="15.24" x2="1.27" y2="15.24" width="0.8128" layer="16"/>
 </signal>
 <signal name="N$2">
@@
 <contactref element="R2" pad="1"/>
 <contactref element="U1" pad="3"/>
-<wire x1="0" y1="12.7" x2="25.4" y2="12.7" width="0.8128" layer="16"/>
-<wire x1="4.064" y1="14.92" x2="2.728" y2="14.92" width="0.4064" layer="1"/>
-<wire x1="2.728" y1="14.92" x2="2.286" y2="14.478" width="0.4064" layer="1"/>
-<wire x1="2.286" y1="14.478" x2="2.286" y2="13.208" width="0.4064" layer="1"/>
-<wire x1="2.286" y1="13.208" x2="1.778" y2="12.7" width="0.4064" layer="1"/>
-<wire x1="1.778" y1="12.7" x2="0" y2="12.7" width="0.4064" layer="1"/>
+<wire x1="1.27" y1="12.7" x2="24.13" y2="12.7" width="0.8128" layer="16"/>
+<wire x1="4.064" y1="14.92" x2="2.982" y2="14.92" width="0.4064" layer="1"/>
+<wire x1="2.982" y1="14.92" x2="2.54" y2="14.478" width="0.4064" layer="1"/>
+<wire x1="2.54" y1="14.478" x2="2.54" y2="13.208" width="0.4064" layer="1"/>
+<wire x1="2.54" y1="13.208" x2="2.032" y2="12.7" width="0.4064" layer="1"/>
+<wire x1="2.032" y1="12.7" x2="1.27" y2="12.7" width="0.4064" layer="1"/>
 <wire x1="8.255" y1="13.8938" x2="8.255" y2="15.367" width="0.4064" layer="1"/>
 <wire x1="8.255" y1="15.367" x2="7.874" y2="15.748" width="0.4064" layer="1"/>
@@
 <contactref element="R1" pad="1"/>
 <contactref element="U1" pad="6"/>
-<wire x1="25.4" y1="10.16" x2="0" y2="10.16" width="0.8128" layer="16"/>
+<wire x1="24.13" y1="10.16" x2="1.27" y2="10.16" width="0.8128" layer="16"/>
 <wire x1="8.255" y1="8.9662" x2="8.255" y2="7.493" width="0.4064" layer="1"/>
 <wire x1="8.255" y1="7.493" x2="7.874" y2="7.112" width="0.4064" layer="1"/>
 <wire x1="7.874" y1="7.112" x2="5.4" y2="7.112" width="0.4064" layer="1"/>
 <wire x1="5.4" y1="7.112" x2="4.064" y2="8.448" width="0.4064" layer="1"/>
-<wire x1="4.064" y1="8.448" x2="2.728" y2="8.448" width="0.4064" layer="1"/>
-<wire x1="2.728" y1="8.448" x2="2.286" y2="8.89" width="0.4064" layer="1"/>
-<wire x1="2.286" y1="8.89" x2="2.286" y2="9.906" width="0.4064" layer="1"/>
-<wire x1="2.286" y1="9.906" x2="2.032" y2="10.16" width="0.4064" layer="1"/>
-<wire x1="2.032" y1="10.16" x2="0" y2="10.16" width="0.4064" layer="1"/>
+<wire x1="4.064" y1="8.448" x2="2.982" y2="8.448" width="0.4064" layer="1"/>
+<wire x1="2.982" y1="8.448" x2="2.54" y2="8.89" width="0.4064" layer="1"/>
+<wire x1="2.54" y1="8.89" x2="2.54" y2="9.906" width="0.4064" layer="1"/>
+<wire x1="2.54" y1="9.906" x2="2.286" y2="10.16" width="0.4064" layer="1"/>
+<wire x1="2.286" y1="10.16" x2="1.27" y2="10.16" width="0.4064" layer="1"/>
 </signal>
 <signal name="N$7">
@@
 <vertex x="-1.27" y="18.288"/>
 </polygon>
-<wire x1="0" y1="5.08" x2="1.27" y2="5.08" width="0.8128" layer="1"/>
-<wire x1="25.4" y1="5.08" x2="24.13" y2="5.08" width="0.8128" layer="1"/>
+<wire x1="1.27" y1="5.08" x2="5.08" y2="5.08" width="0.8128" layer="1"/>
+<wire x1="24.13" y1="5.08" x2="23.622" y2="4.064" width="0.8128" layer="1"/>
+<wire x1="24.13" y1="5.08" x2="23.622" y2="6.096" width="0.8128" layer="1"/>
+<wire x1="12.446" y1="3.976" x2="23.622" y2="4.064" width="0" layer="19" extent="1-1"/>
+<wire x1="5.08" y1="5.08" x2="9.704" y2="4.802" width="0" layer="19" extent="1-1"/>
 </signal>
 <signal name="12V">
@@
 <contactref element="J4" pad="1"/>
 <contactref element="J5" pad="1"/>
-<wire x1="15.442" y1="1.802" x2="9.45" y2="1.802" width="0.8128" layer="1"/>
-<wire x1="0" y1="2.54" x2="0.738" y2="1.802" width="0.8128" layer="1"/>
-<wire x1="0.738" y1="1.802" x2="9.45" y2="1.802" width="0.8128" layer="1"/>
-<wire x1="25.4" y1="2.54" x2="24.662" y2="1.802" width="0.8128" layer="1"/>
-<wire x1="24.662" y1="1.802" x2="15.442" y2="1.802" width="0.8128" layer="1"/>
+<wire x1="15.442" y1="1.802" x2="9.704" y2="1.802" width="0.8128" layer="1"/>
+<wire x1="1.27" y1="2.54" x2="2.262" y2="1.802" width="0.8128" layer="1"/>
+<wire x1="2.262" y1="1.802" x2="9.704" y2="1.802" width="0.8128" layer="1"/>
+<wire x1="24.13" y1="2.54" x2="23.138" y2="1.802" width="0.8128" layer="1"/>
+<wire x1="23.138" y1="1.802" x2="15.442" y2="1.802" width="0.8128" layer="1"/>
 </signal>
 <signal name="3.3V">
@@
 <contactref element="C1" pad="1"/>
 <contactref element="U1" pad="8"/>
-<wire x1="0" y1="7.62" x2="5.842" y2="7.62" width="0.8128" layer="16"/>
+<wire x1="1.27" y1="7.62" x2="5.842" y2="7.62" width="0.8128" layer="16"/>
 <contactref element="R4" pad="3"/>
 <wire x1="5.842" y1="7.62" x2="10.8966" y2="7.62" width="0.8128" layer="16"/>
 <wire x1="10.8966" y1="7.62" x2="18.034" y2="7.62" width="0.8128" layer="16"/>
-<wire x1="18.034" y1="7.62" x2="25.4" y2="7.62" width="0.8128" layer="16"/>
+<wire x1="18.034" y1="7.62" x2="24.13" y2="7.62" width="0.8128" layer="16"/>
 <wire x1="4.064" y1="13.02" x2="4.064" y2="10.348" width="0.4064" layer="1"/>
 <wire x1="4.064" y1="10.348" x2="5.4" y2="10.348" width="0.4064" layer="1"/>
@@
 <via x="10.795" y="6.731" extent="1-16" drill="0.6"/>
 <wire x1="10.795" y1="6.731" x2="10.8966" y2="7.62" width="0.4064" layer="16"/>
-<wire x1="10.795" y1="6.731" x2="12.192" y2="5.676" width="0.4064" layer="1"/>
+<wire x1="10.795" y1="6.731" x2="12.446" y2="5.676" width="0.4064" layer="1"/>
 <via x="18.288" y="6.35" extent="1-16" drill="0.6"/>
 <wire x1="18.288" y1="6.35" x2="18.288" y2="7.366" width="0.4064" layer="16"/>
@@
 <wire x1="21.806" y1="7.662" x2="18.288" y2="7.662" width="0.4064" layer="1"/>
 </signal>
+<signal name="N$4">
+<via x="25.4" y="15.24" extent="1-16" drill="0.6" shape="square"/>
+</signal>
+<signal name="N$5">
+<via x="25.4" y="12.7" extent="1-16" drill="0.6" shape="square"/>
+</signal>
+<signal name="N$6">
+<via x="25.4" y="10.16" extent="1-16" drill="0.6" shape="square"/>
+</signal>
+<signal name="N$9">
+<via x="25.4" y="7.62" extent="1-16" drill="0.6" shape="square"/>
+</signal>
+<signal name="N$10">
+<via x="25.4" y="5.08" extent="1-16" drill="0.6" shape="square"/>
+</signal>
+<signal name="N$11">
+<via x="25.4" y="2.54" extent="1-16" drill="0.6" shape="square"/>
+</signal>
+<signal name="N$12">
+<via x="0" y="15.24" extent="1-16" drill="0.6" shape="square"/>
+</signal>
+<signal name="N$13">
+<via x="0" y="12.7" extent="1-16" drill="0.6" shape="square"/>
+</signal>
+<signal name="N$14">
+<via x="0" y="10.16" extent="1-16" drill="0.6" shape="square"/>
+</signal>
+<signal name="N$15">
+<via x="0" y="7.62" extent="1-16" drill="0.6" shape="square"/>
+</signal>
+<signal name="N$16">
+<via x="0" y="5.08" extent="1-16" drill="0.6" shape="square"/>
+</signal>
+<signal name="N$17">
+<via x="0" y="2.54" extent="1-16" drill="0.6" shape="square"/>
+</signal>
 </signals>
