File: modules/ext_i2c.sch (EAGLE design)
At the start: 11 parts, among them J1 MOLEX_MINILITE_TRAP_2, J2 MOLEX_MINILITE_TRAP_2, J3 MOLEX_MINILITE_TRAP_2, J4 1X06_HEADER_L1X06_EDGE_L, J5 1X06_HEADER_R1X06_EDGE_R, U1 P82B715D

Commit message: Minor changes to cellar controller. Rework of ext_i2c board
Changed lines of the file:
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@@
 <layer number="230" name="230bmp" color="7" fill="1" visible="yes" active="yes"/>
 <layer number="231" name="231bmp" color="7" fill="1" visible="yes" active="yes"/>
+<layer number="232" name="Eagle3D_PG2" color="7" fill="1" visible="no" active="no"/>
+<layer number="233" name="Eagle3D_PG3" color="7" fill="1" visible="no" active="no"/>
 <layer number="248" name="Housing" color="7" fill="1" visible="yes" active="yes"/>
 <layer number="249" name="Edge" color="7" fill="1" visible="yes" active="yes"/>
@@
 <segment>
 <pinref part="U1" gate="A" pin="LX"/>
-<wire x1="68.58" y1="76.2" x2="68.58" y2="55.88" width="0.1524" layer="91"/>
+<wire x1="68.58" y1="73.66" x2="68.58" y2="55.88" width="0.1524" layer="91"/>
 <pinref part="R3" gate="G$1" pin="2"/>
 <wire x1="68.58" y1="55.88" x2="86.36" y2="55.88" width="0.1524" layer="91"/>
@@
 <wire x1="68.58" y1="53.34" x2="78.74" y2="53.34" width="0.1524" layer="91"/>
 <wire x1="78.74" y1="53.34" x2="88.9" y2="53.34" width="0.1524" layer="91"/>
-<wire x1="78.74" y1="76.2" x2="78.74" y2="53.34" width="0.1524" layer="91"/>
+<wire x1="78.74" y1="73.66" x2="78.74" y2="53.34" width="0.1524" layer="91"/>
 <pinref part="R4" gate="G$1" pin="2"/>
 <junction x="78.74" y="53.34"/>
@@
 </segment>
 <segment>
-<wire x1="83.82" y1="81.28" x2="73.66" y2="81.28" width="0.1524" layer="91"/>
+<wire x1="83.82" y1="78.74" x2="73.66" y2="78.74" width="0.1524" layer="91"/>
 <pinref part="SUPPLY6" gate="G$1" pin="3.3V"/>
-<wire x1="73.66" y1="81.28" x2="73.66" y2="86.36" width="0.1524" layer="91"/>
+<wire x1="73.66" y1="78.74" x2="73.66" y2="86.36" width="0.1524" layer="91"/>
 <pinref part="R3" gate="G$1" pin="3"/>
-<junction x="73.66" y="81.28"/>
+<junction x="73.66" y="78.74"/>
 <pinref part="R4" gate="G$1" pin="3"/>
 </segment>
