File: cellar/CellarControl.brd (EAGLE design)
At the start: 61 x 50.8 mm, 34 parts, among them J1 MOLEX_MINILITE_TRAP_2, J2 MOLEX_MINILITE_TRAP_2, J3 MOLEX_MINILITE_TRAP_2, K1 LTV817, T1 BC817, U1 P82B715D

Commit message: Completed Cellar Controller
Parts:
- removed J3: MOLEX_MINILITE_TRAP_2, Puffin:MOLEX_MINILITE_TRAP_2
- S1, S2, S3: value SWITCH-MOMENTARY-2PTH -> SWITCH_MOMENT; device SparkFun-Electromechanical:TACTILE-PTH -> Puffin:SWITCH_MOMENT_6MM
- moved ST2 6.99 mm to (57.1, 10.8)
- moved J2 6.36 mm to (56.4, 33.0), flipped to the top, turned to 0 degrees
- moved S2 3.88 mm to (21.3, 21.0)
- moved S3 3.88 mm to (13.7, 21.0)
- moved S1 3.88 mm to (28.9, 21.0)
- moved R7 2.79 mm to (43.2, 45.4), turned to 0 degrees
- moved R6 2.74 mm to (43.2, 35.2), turned to 0 degrees
- moved RG1 2.54 mm to (47.0, 14.0)
- moved SJ1 2.03 mm to (41.3, 47.6)
- moved SJ2 2.03 mm to (41.3, 32.9)
- moved U$6 1.14 mm to (5.59, 45.5)
- moved R4 0.99 mm to (39.4, 35.2)
- moved R5 0.90 mm to (39.4, 45.4)
- moved U$2 0.57 mm to (5.59, 5.33)
- moved U$4 0.36 mm to (55.6, 5.33)
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Connections:
- removed net N$19: J3.1, RLY1.4
- removed net N$21: J3.2, RLY1.8
- net 12V: now also RLY1.4
- net GND: now also S1.3, S1.4, S2.3, S2.4, S3.3, S3.4; no longer S1.1, S2.1, S3.1
- net N$1: now also RLY1.8
- net N$10: now also S2.1, S2.2; no longer S2.3
- net N$11: now also S3.1, S3.2; no longer S3.3
- net N$9: now also S1.1, S1.2; no longer S1.3
Routing:
- net N$19: track 19.9 -> 0.00 mm
- net 12V: track 65.4 -> 77.6 mm
- net N$21: track 8.88 -> 0.00 mm
- net N$18: track 18.1 -> 23.0 mm, vias 1 -> 2
- net N$1: track 9.88 -> 14.6 mm
- net 3.3V: track 80.5 -> 85.2 mm
- net VSEL: track 39.0 -> 42.7 mm, vias 2 -> 0
- net SDA: track 35.9 -> 34.6 mm
- net SCL: track 38.4 -> 37.0 mm
- net 5V: track 67.9 -> 69.2 mm
- net N$9: track 6.08 -> 4.84 mm
- net N$2: track 4.18 -> 5.25 mm
- net N$6: track 28.6 -> 28.0 mm
Other:
- board text added: "3V3"
- board text added: "500"
- board text added: "5V"

Commit message: Minor changes to cellar controller. Rework of ext_i2c board
Other:
- board text removed: "RELAY2"
Changed lines of the file:
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@@
 <text x="59.2455" y="38.9255" size="1.016" layer="22" font="vector" ratio="15" rot="MR0">PAIR1</text>
 <text x="59.2455" y="32.5755" size="1.016" layer="22" font="vector" ratio="15" rot="MR0">PAIR2</text>
-<text x="44.323" y="7.493" size="1.016" layer="22" font="vector" ratio="15" rot="MR180">RELAY2</text>
 <text x="50.927" y="46.228" size="0.8128" layer="21" font="vector" ratio="15">0</text>
 <text x="46.9265" y="46.228" size="0.8128" layer="21" font="vector" ratio="15">1K</text>
@@
 <wire x1="42.164" y1="33.02" x2="44.45" y2="33.02" width="0.4064" layer="1"/>
 <via x="44.45" y="33.02" extent="1-16" drill="0.6"/>
-<wire x1="44.45" y1="33.02" x2="49.53" y2="33.02" width="0.4064" layer="16"/>
-<wire x1="49.53" y1="33.02" x2="50.165" y2="32.385" width="0.4064" layer="16"/>
-<via x="50.165" y="32.385" extent="1-16" drill="0.6"/>
-<wire x1="50.165" y1="32.385" x2="51.03" y2="31.52" width="0.4064" layer="1"/>
 <wire x1="51.03" y1="31.52" x2="53.288" y2="31.52" width="0.4064" layer="1"/>
-<wire x1="49.4385" y1="38.3075" x2="49.4385" y2="33.1115" width="0.4064" layer="1"/>
-<wire x1="49.4385" y1="33.1115" x2="50.165" y2="32.385" width="0.4064" layer="1"/>
 <wire x1="41.91" y1="37.8587" x2="42.28" y2="35.2425" width="0.4064" layer="1"/>
 <wire x1="42.164" y1="33.02" x2="42.28" y2="35.2425" width="0.4064" layer="1"/>
+<wire x1="44.45" y1="33.02" x2="49.53" y2="33.02" width="0.4064" layer="16"/>
+<wire x1="49.53" y1="33.02" x2="50.292" y2="32.258" width="0.4064" layer="16"/>
+<via x="50.292" y="32.258" extent="1-16" drill="0.6"/>
+<wire x1="50.292" y1="32.258" x2="51.03" y2="31.52" width="0.4064" layer="1"/>
+<wire x1="49.4385" y1="38.3075" x2="49.4385" y2="33.1115" width="0.4064" layer="1"/>
+<wire x1="49.4385" y1="33.1115" x2="50.292" y2="32.258" width="0.4064" layer="1"/>
 </signal>
 <signal name="VSEL">
@@
 </signal>
 <signal name="N$20">
-<via x="50.165" y="32.385" extent="1-16" drill="0.6"/>
 </signal>
 </signals>

Commit message: Gate 4, and misc updates
Connections:
- net N$17 renamed LCL
- net N$18 renamed LDA
Changed lines of the file:
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@@
 <wire x1="23.8125" y1="10.16" x2="24.881" y2="10.16" width="0.4064" layer="1"/>
 </signal>
-<signal name="N$17">
+<signal name="LCL">
 <contactref element="U1" pad="2"/>
 <contactref element="SJ1" pad="2"/>
@@
 <wire x1="46.7885" y1="47.625" x2="42.037" y2="47.625" width="0.4064" layer="1"/>
 </signal>
-<signal name="N$18">
+<signal name="LDA">
 <contactref element="U1" pad="7"/>
 <contactref element="SJ2" pad="2"/>
