File: cellar/CellarControl.sch (EAGLE design)
At the start: 30 parts, among them J1 MOLEX_MINILITE_TRAP_2, J2 MOLEX_MINILITE_TRAP_2, J3 MOLEX_MINILITE_TRAP_2, K1 LTV817, T1 BC817, U1 P82B715D

Commit message: Completed Cellar Controller
Parts:
- removed J3: MOLEX_MINILITE_TRAP_2, Puffin:MOLEX_MINILITE_TRAP_2
- S1, S2, S3: value SWITCH-MOMENTARY-2PTH -> SWITCH_MOMENT; device SparkFun-Electromechanical:SWITCH-MOMENTARY-2PTH -> Puffin:SWITCH_MOMENT
Connections:
- removed net N$19: J3.1, RLY1.C1
- removed net N$21: J3.2, RLY1.NO1
- net 12V: now also RLY1.C1
- net GND: now also S1.2, S2.2, S3.2; no longer S1.1, S2.1, S3.1
- net N$1: now also RLY1.NO1
- net N$10: now also S2.1; no longer S2.2
- net N$11: now also S3.1; no longer S3.2
- net N$9: now also S1.1; no longer S1.2
Other:
- note removed: "C NO"
Changed lines of the file:
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@@
 <part name="GND8" library="SparkFun-Aesthetics" deviceset="GND" device=""/>
 <part name="SUPPLY3" library="SparkFun-Aesthetics" deviceset="3.3V" device=""/>
-<part name="S1" library="SparkFun-Electromechanical" deviceset="SWITCH-MOMENTARY-2" device="PTH"/>
-<part name="S2" library="SparkFun-Electromechanical" deviceset="SWITCH-MOMENTARY-2" device="PTH"/>
-<part name="S3" library="SparkFun-Electromechanical" deviceset="SWITCH-MOMENTARY-2" device="PTH"/>
 <part name="GND1" library="SparkFun-Aesthetics" deviceset="GND" device=""/>
 <part name="SUPPLY5" library="SparkFun-Aesthetics" deviceset="5V" device=""/>
@@
 <part name="T1" library="Puffin" deviceset="BC817" device=""/>
 <part name="K1" library="Puffin" deviceset="LTV817" device=""/>
-<part name="J3" library="Puffin" deviceset="MOLEX_MINILITE_TRAP_2" device=""/>
 <part name="R8" library="Puffin" deviceset="POT_3MM" device=""/>
 <part name="R9" library="Puffin" deviceset="POT_3MM" device=""/>
@@
 <part name="RG1" library="Puffin" deviceset="MURATA_REG" device=""/>
 <part name="D2" library="SparkFun-LED" deviceset="LED" device="3MM"/>
+<part name="S1" library="Puffin" deviceset="SWITCH_MOMENT" device=""/>
+<part name="S2" library="Puffin" deviceset="SWITCH_MOMENT" device=""/>
+<part name="S3" library="Puffin" deviceset="SWITCH_MOMENT" device=""/>
 </parts>
 <sheets>
@@
 <text x="230.124" y="163.068" size="1.778" layer="94">12Vin</text>
 <text x="230.124" y="157.988" size="1.778" layer="94">Pump</text>
-<text x="227.33" y="177.038" size="1.778" layer="94">C
-NO</text>
 <text x="237.744" y="94.488" size="1.778" layer="94">Pair 1</text>
 <text x="237.744" y="84.328" size="1.778" layer="94">Pair 2</text>
-<text x="120.65" y="82.296" size="1.778" layer="94">Home</text>
-<text x="121.158" y="74.676" size="1.778" layer="94">Up</text>
-<text x="120.65" y="66.548" size="1.778" layer="94">Down</text>
+<text x="113.792" y="82.296" size="1.778" layer="94">Home</text>
+<text x="114.808" y="74.676" size="1.778" layer="94">Up</text>
+<text x="113.538" y="67.056" size="1.778" layer="94">Down</text>
 </plain>
 <instances>
@@
 <instance part="FRAME1" gate="G$2" x="147.32" y="0"/>
 <instance part="SF1" gate="G$1" x="25.4" y="132.08" smashed="yes">
-<attribute name="NAME" x="15.748" y="143.002" size="1.778" layer="94"/>
+<attribute name="NAME" x="18.288" y="143.002" size="1.778" layer="94"/>
 </instance>
 <instance part="SC1" gate="G$1" x="86.36" y="121.92"/>
@@
 <instance part="GND8" gate="1" x="223.52" y="78.74"/>
 <instance part="SUPPLY3" gate="G$1" x="40.64" y="147.32"/>
-<instance part="S1" gate="G$1" x="119.38" y="66.04" smashed="yes" rot="MR0">
-<attribute name="NAME" x="116.332" y="66.548" size="1.778" layer="95" rot="MR0"/>
-</instance>
-<instance part="S2" gate="G$1" x="119.38" y="73.66" smashed="yes" rot="MR0">
-<attribute name="NAME" x="116.586" y="74.422" size="1.778" layer="95" rot="MR0"/>
-</instance>
-<instance part="S3" gate="G$1" x="119.38" y="81.28" smashed="yes" rot="MR0">
-<attribute name="NAME" x="116.332" y="82.042" size="1.778" layer="95" rot="MR0"/>
-</instance>
 <instance part="GND1" gate="1" x="127" y="60.96"/>
 <instance part="SUPPLY5" gate="G$1" x="63.5" y="157.48"/>
@@
 <instance part="T1" gate="G$1" x="170.18" y="134.62"/>
 <instance part="K1" gate="G$1" x="139.7" y="137.16"/>
-<instance part="J3" gate="G$1" x="220.98" y="177.8" rot="MR0"/>
 <instance part="R8" gate="G$1" x="205.74" y="101.6"/>
 <instance part="R9" gate="G$1" x="198.12" y="101.6"/>
@@
 <instance part="RG1" gate="RG$1" x="149.86" y="172.72"/>
 <instance part="D2" gate="G$1" x="43.18" y="88.9"/>
+<instance part="S1" gate="G$1" x="119.38" y="66.04" smashed="yes">
+<attribute name="NAME" x="122.174" y="66.802" size="1.778" layer="95"/>
+</instance>
+<instance part="S2" gate="G$1" x="119.38" y="73.66" smashed="yes">
+<attribute name="NAME" x="122.174" y="74.422" size="1.778" layer="95"/>
+</instance>
+<instance part="S3" gate="G$1" x="119.38" y="81.28" smashed="yes">
+<attribute name="NAME" x="122.174" y="82.042" size="1.778" layer="95"/>
+</instance>
 </instances>
 <busses>
@@
 <pinref part="GND1" gate="1" pin="GND"/>
 <wire x1="127" y1="81.28" x2="127" y2="73.66" width="0.1524" layer="91"/>
-<pinref part="S3" gate="G$1" pin="1"/>
 <wire x1="127" y1="73.66" x2="127" y2="66.04" width="0.1524" layer="91"/>
 <wire x1="127" y1="66.04" x2="127" y2="63.5" width="0.1524" layer="91"/>
 <wire x1="124.46" y1="81.28" x2="127" y2="81.28" width="0.1524" layer="91"/>
-<pinref part="S2" gate="G$1" pin="1"/>
 <wire x1="124.46" y1="73.66" x2="127" y2="73.66" width="0.1524" layer="91"/>
-<pinref part="S1" gate="G$1" pin="1"/>
 <wire x1="124.46" y1="66.04" x2="127" y2="66.04" width="0.1524" layer="91"/>
 <junction x="127" y="73.66"/>
 <junction x="127" y="66.04"/>
+<pinref part="S1" gate="G$1" pin="2"/>
+<pinref part="S2" gate="G$1" pin="2"/>
+<pinref part="S3" gate="G$1" pin="2"/>
 </segment>
 <segment>
@@
 <wire x1="218.44" y1="165.1" x2="203.2" y2="165.1" width="0.1524" layer="91"/>
 <junction x="203.2" y="165.1"/>
+<wire x1="203.2" y1="165.1" x2="177.8" y2="165.1" width="0.1524" layer="91"/>
+<wire x1="177.8" y1="165.1" x2="177.8" y2="147.32" width="0.1524" layer="91"/>
+<pinref part="RLY1" gate="G$1" pin="C1"/>
+<wire x1="177.8" y1="147.32" x2="182.88" y2="147.32" width="0.1524" layer="91"/>
 </segment>
 <segment>
@@
 <wire x1="104.14" y1="104.14" x2="106.68" y2="104.14" width="0.1524" layer="91"/>
 <wire x1="106.68" y1="104.14" x2="106.68" y2="66.04" width="0.1524" layer="91"/>
-<pinref part="S1" gate="G$1" pin="2"/>
 <wire x1="106.68" y1="66.04" x2="114.3" y2="66.04" width="0.1524" layer="91"/>
+<pinref part="S1" gate="G$1" pin="1"/>
 </segment>
 </net>
@@
 <wire x1="104.14" y1="109.22" x2="109.22" y2="109.22" width="0.1524" layer="91"/>
 <wire x1="109.22" y1="109.22" x2="109.22" y2="73.66" width="0.1524" layer="91"/>
-<pinref part="S2" gate="G$1" pin="2"/>
 <wire x1="109.22" y1="73.66" x2="114.3" y2="73.66" width="0.1524" layer="91"/>
+<pinref part="S2" gate="G$1" pin="1"/>
 </segment>
 </net>
@@
 <pinref part="SC1" gate="G$1" pin="D4"/>
 <wire x1="104.14" y1="114.3" x2="111.76" y2="114.3" width="0.1524" layer="91"/>
-<pinref part="S3" gate="G$1" pin="2"/>
 <wire x1="111.76" y1="114.3" x2="111.76" y2="81.28" width="0.1524" layer="91"/>
 <wire x1="111.76" y1="81.28" x2="114.3" y2="81.28" width="0.1524" layer="91"/>
+<pinref part="S3" gate="G$1" pin="1"/>
 </segment>
 </net>
@@
 <wire x1="220.98" y1="93.98" x2="226.06" y2="93.98" width="0.1524" layer="91"/>
 <pinref part="R7" gate="G$1" pin="1"/>
-<wire x1="193.04" y1="106.68" x2="193.04" y2="101.6" width="0.1524" layer="91"/>
+<wire x1="193.04" y1="106.68" x2="193.04" y2="99.06" width="0.1524" layer="91"/>
 <pinref part="R9" gate="G$1" pin="2"/>
-<junction x="193.04" y="101.6"/>
-<wire x1="193.04" y1="101.6" x2="193.04" y2="91.44" width="0.1524" layer="91"/>
+<junction x="193.04" y="99.06"/>
+<wire x1="193.04" y1="99.06" x2="193.04" y2="91.44" width="0.1524" layer="91"/>
 </segment>
 </net>
@@
 <wire x1="220.98" y1="86.36" x2="226.06" y2="86.36" width="0.1524" layer="91"/>
 <pinref part="R6" gate="G$1" pin="1"/>
-<wire x1="200.66" y1="106.68" x2="200.66" y2="101.6" width="0.1524" layer="91"/>
+<wire x1="200.66" y1="106.68" x2="200.66" y2="99.06" width="0.1524" layer="91"/>
 <pinref part="R8" gate="G$1" pin="2"/>
-<junction x="200.66" y="101.6"/>
-<wire x1="200.66" y1="101.6" x2="200.66" y2="88.9" width="0.1524" layer="91"/>
-</segment>
-</net>
-<net name="N$21" class="0">
-<segment>
-<pinref part="RLY1" gate="G$1" pin="NO1"/>
-<wire x1="182.88" y1="157.48" x2="180.34" y2="157.48" width="0.1524" layer="91"/>
-<wire x1="180.34" y1="157.48" x2="180.34" y2="177.8" width="0.1524" layer="91"/>
-<pinref part="J3" gate="G$1" pin="2"/>
-<wire x1="180.34" y1="177.8" x2="215.9" y2="177.8" width="0.1524" layer="91"/>
-</segment>
-</net>
-<net name="N$19" class="0">
-<segment>
-<pinref part="RLY1" gate="G$1" pin="C1"/>
-<wire x1="182.88" y1="147.32" x2="175.26" y2="147.32" width="0.1524" layer="91"/>
-<wire x1="175.26" y1="147.32" x2="175.26" y2="180.34" width="0.1524" layer="91"/>
-<pinref part="J3" gate="G$1" pin="1"/>
-<wire x1="175.26" y1="180.34" x2="215.9" y2="180.34" width="0.1524" layer="91"/>
+<junction x="200.66" y="99.06"/>
+<wire x1="200.66" y1="99.06" x2="200.66" y2="88.9" width="0.1524" layer="91"/>
 </segment>
 </net>
@@
 <junction x="200.66" y="116.84"/>
 <pinref part="R9" gate="G$1" pin="3"/>
-<wire x1="198.12" y1="106.68" x2="198.12" y2="116.84" width="0.1524" layer="91"/>
+<wire x1="198.12" y1="104.14" x2="198.12" y2="116.84" width="0.1524" layer="91"/>
 <pinref part="R8" gate="G$1" pin="3"/>
-<wire x1="205.74" y1="106.68" x2="205.74" y2="116.84" width="0.1524" layer="91"/>
+<wire x1="205.74" y1="104.14" x2="205.74" y2="116.84" width="0.1524" layer="91"/>
 <junction x="198.12" y="116.84"/>
 <junction x="205.74" y="116.84"/>
@@
 <pinref part="RLY1" gate="G$1" pin="NO2"/>
 <pinref part="ST2" gate="G$1" pin="1"/>
-<wire x1="198.12" y1="157.48" x2="218.44" y2="157.48" width="0.1524" layer="91"/>
+<wire x1="198.12" y1="157.48" x2="200.66" y2="157.48" width="0.1524" layer="91"/>
+<wire x1="200.66" y1="157.48" x2="218.44" y2="157.48" width="0.1524" layer="91"/>
+<wire x1="200.66" y1="157.48" x2="200.66" y2="162.56" width="0.1524" layer="91"/>
+<pinref part="RLY1" gate="G$1" pin="NO1"/>
+<wire x1="182.88" y1="157.48" x2="180.34" y2="157.48" width="0.1524" layer="91"/>
+<wire x1="200.66" y1="162.56" x2="180.34" y2="162.56" width="0.1524" layer="91"/>
+<wire x1="180.34" y1="162.56" x2="180.34" y2="157.48" width="0.1524" layer="91"/>
+<junction x="200.66" y="157.48"/>
 </segment>
 </net>
@@
 </schematic>
 </drawing>
-<compatibility>
-<note version="6.3" minversion="6.2.2" severity="warning">
-Since Version 6.2.2 text objects can contain more than one line,
-which will not be processed correctly with this version.
-</note>
-</compatibility>
 </eagle>

Commit message: Gate 4, and misc updates
Connections:
- net N$17 renamed LCL
- net N$18 renamed LDA
Changed lines of the file:
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@@
 </segment>
 </net>
-<net name="N$17" class="0">
+<net name="LCL" class="0">
 <segment>
 <wire x1="193.04" y1="91.44" x2="220.98" y2="91.44" width="0.1524" layer="91"/>
@@
 </segment>
 </net>
-<net name="N$18" class="0">
+<net name="LDA" class="0">
 <segment>
 <wire x1="200.66" y1="88.9" x2="220.98" y2="88.9" width="0.1524" layer="91"/>
