File: gate/gate4.sch (EAGLE design)
At the start: 32 parts, among them J1 MOLEX_MINILITE_TRAP_2, J2 MOLEX_MINILITE_TRAP_2, J3 MOLEX_MINILITE_TRAP_2, J4 MOLEX_MINILITE_TRAP_2, J8 MOLEX_MINILITE_TRAP_2, J9 MOLEX_MINILITE_TRAP_2, U1 SN75468

Commit message: Gate 4, and misc updates
Parts:
- removed J10: (no value), SparkFun-Connectors:M07
- removed JP0, JP1: JUMPER-PAD-3-2OF3_NC_BY_TRACE_SMALL, SparkFun-Passives:JUMPER-PAD-3-2OF3_NC_BY_TRACE_SMALL
- added JP7, JP8: JUMPER-PAD-2-NOYES_SILK, SparkFun-Passives:JUMPER-PAD-2-NOYES_SILK
- added SJ1: (no value), jumper:SJ
- added ST5: (no value), Puffin:SCREWTERM_2
- J5: device SparkFun-Connectors:M04X2 -> SparkFun-Connectors:M07
- J9: value MOLEX_MINILITE_TRAP_2 -> (none); device Puffin:MOLEX_MINILITE_TRAP_2 -> SparkFun-Connectors:M04PTH
- JP2, JP3, JP4, JP5, JP6: value JUMPER-PAD-3-2OF3_NC_BY_TRACE_SMALL -> JUMPER-PAD-2-NOYES_SILK; device SparkFun-Passives:JUMPER-PAD-3-2OF3_NC_BY_TRACE_SMALL -> SparkFun-Passives:JUMPER-PAD-2-NOYES_SILK
Connections:
- removed net D0: E1.D0, JP0.3
- removed net D1: E1.D1, JP1.3
- removed net D2: E1.D2, JP2.3
- removed net D3: E1.D3, JP3.3
- removed net D4: E1.D4, JP4.3
- removed net D5: E1.D5, JP5.3
- removed net D6: E1.D6, JP6.3
- removed net J0: J10.1, JP0.2
- removed net J1: J10.2, JP1.2
- removed net J2: J10.3, JP2.2
- removed net J3: J10.4, JP3.2
- removed net J4: J10.5, JP4.2
- removed net J5: J10.6, JP5.2
- removed net J6: J10.7, JP6.2
- new net N$22: R2.R2, U1.OUT2
- new net N$30: E1.D0, J5.7, JP8.2
- new net N$31: E1.D1, J5.6, JP7.2
- new net N$32: E1.D2, J5.5, JP6.2
- new net N$36: E1.D4, J5.3, JP4.2
- new net N$37: E1.D5, J5.2, JP3.2
- new net N$38: E1.D6, J5.1, JP2.2
- net 3.3V: now also J9.3; no longer J5.5, J5.6
- net 5V: now also J9.2, SJ1.2; no longer J5.3, J5.4, J9.1
- net A0: now also JP8.1; no longer JP0.1
- net A1: now also JP7.1; no longer JP1.1
- net A2: now also JP6.1; no longer JP2.1
- net A3: now also JP5.1; no longer JP3.1
- net A5: now also JP3.1; no longer JP5.1
- net A6: now also JP2.1; no longer JP6.1
- net GND: now also J9.4, ST5.1; no longer J5.7, J5.8, J9.2
- net N$1: now also ST1.2; no longer ST1.1
- net N$23: now also ST1.1; no longer ST1.2
- net N$3: now also R5.P$1; no longer R3.R2
- net N$33: now also R1.R2; no longer R7.P$1
- net N$34: now also E1.D3, J5.4, JP5.2; no longer R6.P$1, U1.OUT2
- net N$35: now also R3.R2; no longer R5.P$1
- net N$4: now also R6.P$1; no longer R2.R2
- net N$5: now also R7.P$1; no longer R1.R2
- net VIN: now also J9.1, SJ1.1, ST5.2; no longer J5.1, J5.2
Other:
- moved on the sheet: J1, J2, J3, J4, J8, R1, R2, R3, R4, R5, R6, R7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
