File: gate/gate5.brd (EAGLE design)
At the start: 44.5 x 94 mm, 32 parts, among them J1 MOLEX_MINILITE_TRAP_2, J2 MOLEX_MINILITE_TRAP_2, J3 MOLEX_MINILITE_TRAP_2, J4 MOLEX_MINILITE_TRAP_2, J5 MOLEX_MINILITE_TRAP_2, U1 SN75468, U2 E0_V005

Commit message: Gate 5 updated, not sure what changed
Parts:
- removed H1, H2, H3, H4: STAND-OFF, SparkFun-Electromechanical:STAND-OFF
- removed R6, R7, R8, R9: 2.2K, SparkFun-Resistors:0603-RES
- removed U$1: PHOTON_SMD, Particle:PHOTON_SMD
- removed U2: E0_V005, Particle:E0
- added M1: ELECTRON, Puffin:ELECTRON
- added RL1, RL2, RL3, RL4: HE3600_RELAY, Puffin:HE3600_RELAY
- added ST2, ST3, ST4, ST5: (no value), Puffin:SCREWTERM_0.2X2
- C1: value (none) -> 470uf
- J6: device SparkFun-Connectors:2X4 -> SparkFun-Connectors:2X8
- R1, R2, R3, R4: value HE3600_RELAY -> 2.2K; device Puffin:HE3600_RELAY -> SparkFun-Resistors:0603-RES
- moved J5 77.7 mm to (39.9, 14.0), turned to 0 degrees
- moved RG2 55.7 mm to (39.4, 27.2)
- moved RG1 55.1 mm to (39.4, 35.6)
- moved SJ1 54.4 mm to (39.4, 39.0)
- moved D5 54.2 mm to (39.4, 42.7)
- moved J6 34.2 mm to (24.1, 55.9), turned to 270 degrees
- moved R4 28.2 mm to (32.9, 50.8)
- moved J4 27.9 mm to (39.9, 50.8)
- moved D4 27.9 mm to (34.3, 50.8), turned to 0 degrees
- moved R1 21.9 mm to (32.9, 81.3)
- moved J1 21.6 mm to (39.9, 81.3)
- moved D1 21.6 mm to (34.3, 81.3), turned to 0 degrees
- moved R5 19.6 mm to (39.4, 41.3), turned to 180 degrees
- moved C1 15.1 mm to (27.9, 19.1), turned to 90 degrees
- moved ST1 14.5 mm to (40.6, 78.7), turned to 90 degrees
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Connections:
- net R6 renamed L6
- removed net N$15: J6.7
- removed net R5: J6.1, U1.12
- removed net R7: J6.5, U1.10
- removed net VBAT: U$1.22
- new net A0: J6.15, M1.A0
- new net A1: J6.13, M1.A1
- new net A2: J6.11, M1.A2
- new net A3: J6.9, M1.A3
- new net A4: J6.7, M1.A4
- new net L5: J6.5, U1.12
- new net L7: J6.1, U1.10
- net 3.3V: now also M1.3V3; no longer J6.6, U$1.24, U2.9
- net 5V: now also J6.2, J6.6, M1.VIN, R1.1, R2.1, R3.1, R4.1, RL1.2, RL2.2, RL3.2, RL4.2; no longer R1.2, R2.2, R3.2, R4.2, R6.1, R7.1, R8.1, R9.1, U$1.1, U2.1
- net D0: now also M1.D0; no longer U$1.13, U2.42
- net D1: now also M1.D1; no longer U$1.14, U2.41
- net D2: now also M1.D2; no longer U$1.15, U2.40
- net D3: now also M1.D3; no longer U$1.16, U2.39
- net D4: now also M1.D4; no longer U$1.17, U2.38
- net D5: now also M1.D5; no longer U$1.18, U2.37
- net D6: now also M1.D6; no longer U$1.19, U2.36
- net GND: now also J6.10, J6.12, J6.14, J6.16, M1.GND, M1.GND@2, ST5.1; no longer J6.8, ST1.1, U$1.2, U$1.21, U2.12, U2.15, U2.18, U2.2, U2.27, U2.34, U2.4, U2.43, U2.51, U2.58, U2.59, U2.60, U2.7
- net N$1: now also R2.2; no longer R6.2
- net N$10: now also RL3.1, ST3.2; no longer R3.1
- net N$11: now also RL4.1, ST4.2; no longer R4.1
- net N$12: now also RL1.4, ST1.1; no longer R1.4
- net N$13: now also RL1.1, ST1.2; no longer R1.1
- net N$14: now also R5.2; no longer R9.2
- net N$2: now also RL4.3; no longer R4.3
- net N$22: now also RL2.3; no longer R2.3
- net N$3: now also R1.2; no longer R5.2
- net N$33: now also RL1.3; no longer R1.3
- net N$35: now also RL3.3; no longer R3.3
- net N$4: now also R3.2; no longer R7.2
- net N$5: now also R4.2; no longer R8.2
- net N$6: now also RL4.4, ST4.1; no longer R4.4
- net N$7: now also RL3.4, ST3.1; no longer R3.4
- net N$8: now also RL2.4, ST2.1; no longer R2.4
- net N$9: now also RL2.1, ST2.2; no longer R2.1
- net VIN: now also J6.8, ST5.2; no longer J6.2, ST1.2
Routing:
- net 3.3V: track 124.3 -> 0.00 mm, vias 2 -> 0
- net D1: track 79.8 -> 38.4 mm, vias 3 -> 0
- net D0: track 82.5 -> 41.5 mm, vias 3 -> 0
- net D2: track 76.2 -> 35.3 mm, vias 3 -> 0
- net D3: track 73.1 -> 32.3 mm, vias 3 -> 0
- net D4: track 69.9 -> 29.2 mm, vias 3 -> 0
- net D5: track 64.6 -> 26.1 mm, vias 3 -> 0
- net D6: track 60.4 -> 23.1 mm, vias 2 -> 0
- net 5V: track 49.9 -> 14.5 mm, vias 3 -> 5
- net L5: track 0.00 -> 27.2 mm
- net A4: track 0.00 -> 26.3 mm
- net A3: track 0.00 -> 26.3 mm
- net A2: track 0.00 -> 26.3 mm
- net A1: track 0.00 -> 26.3 mm
- net A0: track 0.00 -> 26.3 mm
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Other:
- board size 44.5 x 94 mm -> 105 x 101.6 mm
- board text added: "7-36V"
- board text added: "A"
- board text added: "B"
- board text added: "C"
- board text added: "D"
- board text added: "PWR"
- board text removed: "3V3"
- board text removed: "5V"
