File: gate/gate5.sch (EAGLE design)
At the start: 32 parts, among them J1 MOLEX_MINILITE_TRAP_2, J2 MOLEX_MINILITE_TRAP_2, J3 MOLEX_MINILITE_TRAP_2, J4 MOLEX_MINILITE_TRAP_2, J5 MOLEX_MINILITE_TRAP_2, U1 SN75468, U2 E0_V005

Commit message: Gate 5 updated, not sure what changed
Parts:
- removed H1, H2, H3, H4: STAND-OFF, SparkFun-Electromechanical:STAND-OFF
- removed R6, R7, R8, R9: 2.2K, SparkFun-Resistors:RESISTOR0603
- removed U$1: PHOTON_SMD, Particle:PHOTON_SMD
- removed U2: E0_V005, Particle:E0_V005
- added M1: ELECTRON, Puffin:ELECTRON
- added RL1, RL2, RL3, RL4: HE3600_RELAY, Puffin:HE3600_RELAY
- added ST2, ST3, ST4, ST5: (no value), Puffin:SCREWTERM_2
- C1: value (none) -> 470uf
- J6: device SparkFun-Connectors:M04X2 -> SparkFun-Connectors:M08X2
- R1, R2, R3, R4: value HE3600_RELAY -> 2.2K; device Puffin:HE3600_RELAY -> SparkFun-Resistors:RESISTOR0603
Connections:
- net R6 renamed L6
- removed net N$15: J6.7
- removed net R5: J6.1, U1.OUT5
- removed net R7: J6.5, U1.OUT7
- new net A0: J6.15, M1.A0
- new net A1: J6.13, M1.A1
- new net A2: J6.11, M1.A2
- new net A3: J6.9, M1.A3
- new net A4: J6.7, M1.A4
- new net L5: J6.5, U1.OUT5
- new net L7: J6.1, U1.OUT7
- net 3.3V: now also M1.3V3; no longer J6.6, U$1G$1.3V3, U2.3V3
- net 5V: now also J6.2, J6.6, M1.VIN, R1.1, R2.1, R3.1, R4.1, RL1.R1, RL2.R1, RL3.R1, RL4.R1; no longer R1.R1, R2.R1, R3.R1, R4.R1, R6.1, R7.1, R8.1, R9.1, U$1G$1.VIN, U2.VIN
- net D0: now also M1.D0; no longer U$1G$1.D0, U2.D0
- net D1: now also M1.D1; no longer U$1G$1.D1, U2.D1
- net D2: now also M1.D2; no longer U$1G$1.D2, U2.D2
- net D3: now also M1.D3; no longer U$1G$1.D3, U2.D3
- net D4: now also M1.D4; no longer U$1G$1.D4, U2.D4
- net D5: now also M1.D5; no longer U$1G$1.D5, U2.D5
- net D6: now also M1.D6; no longer U$1G$1.D6, U2.D6
- net GND: now also J6.10, J6.12, J6.14, J6.16, M1.GND, M1.GND@2, ST5.1; no longer J6.8, ST1.1, U$1G$1.GND@2, U$1G$1.GND@21, U2.GND@12, U2.GND@15, U2.GND@18, U2.GND@2, U2.GND@27, U2.GND@34, U2.GND@4, U2.GND@43, U2.GND@51, U2.GND@7, U2.GND@PADS
- net N$1: now also R2.2; no longer R6.2
- net N$10: now also RL3.C1, ST3.2; no longer R3.C1
- net N$11: now also RL4.C1, ST4.2; no longer R4.C1
- net N$12: now also RL1.C2, ST1.1; no longer R1.C2
- net N$13: now also RL1.C1, ST1.2; no longer R1.C1
- net N$14: now also R5.2; no longer R9.2
- net N$2: now also RL4.R2; no longer R4.R2
- net N$22: now also RL2.R2; no longer R2.R2
- net N$3: now also R1.2; no longer R5.2
- net N$33: now also RL1.R2; no longer R1.R2
- net N$35: now also RL3.R2; no longer R3.R2
- net N$4: now also R3.2; no longer R7.2
- net N$5: now also R4.2; no longer R8.2
- net N$6: now also RL4.C2, ST4.1; no longer R4.C2
- net N$7: now also RL3.C2, ST3.1; no longer R3.C2
- net N$8: now also RL2.C2, ST2.1; no longer R2.C2
- net N$9: now also RL2.C1, ST2.2; no longer R2.C1
- net VIN: now also J6.8, ST5.2; no longer J6.2, ST1.2
Other:
- moved on the sheet: C1, D1, D2, D3, D4, D5, J1, J2, J3, J4, J5, R5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
